Commit message: Update link2 mesh and ros2_control config.
Switch link2 to glb mesh and drop unused arm_controller entry from ros2_controllers.yaml.

Co-authored-by: Cursor <cursoragent@cursor.com>

File: xacro/panthera_ht.xacro (robot description, xacro)
@@ -77,10 +77,10 @@
       <visual>
         <geometry>
-          <mesh filename="file://$(find panthera_ht_description)/meshes/visual/link2.STL"/>
-        </geometry>
-      </visual>
-      <collision>
-        <geometry>
-          <mesh filename="file://$(find panthera_ht_description)/meshes/visual/link2.STL"/>
+          <mesh filename="file://$(find panthera_ht_description)/meshes/link2.glb"/>
+        </geometry>
+      </visual>
+      <collision>
+        <geometry>
+          <mesh filename="file://$(find panthera_ht_description)/meshes/link2.glb"/>
         </geometry>
       </collision>

Commit message: Sync local Panthera HT description updates.
Include ros2_control/xacro/mesh changes from the deploy workspace before relocating into robot-descriptions-ht.

Co-authored-by: Cursor <cursoragent@cursor.com>

File: xacro/panthera_ht.xacro (robot description, xacro)
@@ -108,10 +108,10 @@
       <visual>
         <geometry>
-          <mesh filename="file://$(find panthera_ht_description)/meshes/visual/link3.STL"/>
-        </geometry>
-      </visual>
-      <collision>
-        <geometry>
-          <mesh filename="file://$(find panthera_ht_description)/meshes/visual/link3.STL"/>
+          <mesh filename="file://$(find panthera_ht_description)/meshes/link3.glb"/>
+        </geometry>
+      </visual>
+      <collision>
+        <geometry>
+          <mesh filename="file://$(find panthera_ht_description)/meshes/link3.glb"/>
         </geometry>
       </collision>
@@ -139,10 +139,10 @@
       <visual>
         <geometry>
-          <mesh filename="file://$(find panthera_ht_description)/meshes/visual/link4.STL"/>
-        </geometry>
-      </visual>
-      <collision>
-        <geometry>
-          <mesh filename="file://$(find panthera_ht_description)/meshes/visual/link4.STL"/>
+          <mesh filename="file://$(find panthera_ht_description)/meshes/link4.glb"/>
+        </geometry>
+      </visual>
+      <collision>
+        <geometry>
+          <mesh filename="file://$(find panthera_ht_description)/meshes/link4.glb"/>
         </geometry>
       </collision>
@@ -170,10 +170,10 @@
       <visual>
         <geometry>
-          <mesh filename="file://$(find panthera_ht_description)/meshes/visual/link5.STL"/>
-        </geometry>
-      </visual>
-      <collision>
-        <geometry>
-          <mesh filename="file://$(find panthera_ht_description)/meshes/visual/link5.STL"/>
+          <mesh filename="file://$(find panthera_ht_description)/meshes/link5.glb"/>
+        </geometry>
+      </visual>
+      <collision>
+        <geometry>
+          <mesh filename="file://$(find panthera_ht_description)/meshes/link5.glb"/>
         </geometry>
       </collision>
@@ -201,10 +201,10 @@
       <visual>
         <geometry>
-          <mesh filename="file://$(find panthera_ht_description)/meshes/visual/link6.STL"/>
-        </geometry>
-      </visual>
-      <collision>
-        <geometry>
-          <mesh filename="file://$(find panthera_ht_description)/meshes/visual/link6.STL"/>
+          <mesh filename="file://$(find panthera_ht_description)/meshes/link6.glb"/>
+        </geometry>
+      </visual>
+      <collision>
+        <geometry>
+          <mesh filename="file://$(find panthera_ht_description)/meshes/link6.glb"/>
         </geometry>
       </collision>

File: xacro/robot.xacro (robot description, xacro)
@@ -1,5 +1,72 @@
 <?xml version="1.0"?>
 <robot name="Panthera HT" xmlns:xacro="http://www.ros.org/wiki/xacro">
+  <!-- `type` follows robot_common_launch conventions (like Tianji):
+       - empty (default): single arm (legacy)
+       - left | right | dual: mount one or two arms on a shared body
+  -->
+  <xacro:arg name="type" default="empty"/>
+  <xacro:arg name="body_xyz" default="0 0 0"/>
+  <xacro:arg name="body_rpy" default="0 0 0"/>
+  <xacro:arg name="left_mount_xyz" default="0 0.35 0"/>
+  <xacro:arg name="left_mount_rpy" default="0 0 0"/>
+  <xacro:arg name="right_mount_xyz" default="0 -0.35 0"/>
+  <xacro:arg name="right_mount_rpy" default="0 0 0"/>
   <xacro:include filename="$(find panthera_ht_description)/xacro/panthera_ht.xacro"/>
-  <xacro:Arm name=""/>
+  <!-- resolve arm composition from `type` (Tianji-style) -->
+  <xacro:property name="_type" value="$(arg type)"/>
+  <xacro:property name="_arm_config" value="single"/>
+  <xacro:if value="${_type == 'left'}">
+    <xacro:property name="_arm_config" value="left"/>
+  </xacro:if>
+  <xacro:if value="${_type == 'right'}">
+    <xacro:property name="_arm_config" value="right"/>
+  </xacro:if>
+  <xacro:if value="${_type == 'dual'}">
+    <xacro:property name="_arm_config" value="dual"/>
+  </xacro:if>
+  <!-- Single arm (legacy): root link is `base_link` -->
+  <xacro:if value="${_arm_config == 'single'}">
+    <xacro:Arm name=""/>
+  </xacro:if>
+  <!-- Left-only / Right-only / Dual arms: mount one or two prefixed arms on a shared body -->
+  <xacro:unless value="${_arm_config == 'single'}">
+    <link name="world"/>
+    <link name="base_link"/>
+    <link name="body_link"/>
+    <link name="left_mount"/>
+    <link name="right_mount"/>
+    <joint name="base_joint" type="fixed">
+      <parent link="world"/>
+      <child link="base_link"/>
+    </joint>
+    <joint name="body_joint" type="fixed">
+      <origin xyz="$(arg body_xyz)" rpy="$(arg body_rpy)"/>
+      <parent link="base_link"/>
+      <child link="body_link"/>
+    </joint>
+    <joint name="left_mount_joint" type="fixed">
+      <origin xyz="$(arg left_mount_xyz)" rpy="$(arg left_mount_rpy)"/>
+      <parent link="body_link"/>
+      <child link="left_mount"/>
+    </joint>
+    <joint name="right_mount_joint" type="fixed">
+      <origin xyz="$(arg right_mount_xyz)" rpy="$(arg right_mount_rpy)"/>
+      <parent link="body_link"/>
+      <child link="right_mount"/>
+    </joint>
+    <xacro:if value="${_arm_config == 'left' or _arm_config == 'dual'}">
+      <xacro:Arm name="left"/>
+      <joint name="left_arm_mount_joint" type="fixed">
+        <parent link="left_mount"/>
+        <child link="left_base_link"/>
+      </joint>
+    </xacro:if>
+    <xacro:if value="${_arm_config == 'right' or _arm_config == 'dual'}">
+      <xacro:Arm name="right"/>
+      <joint name="right_arm_mount_joint" type="fixed">
+        <parent link="right_mount"/>
+        <child link="right_base_link"/>
+      </joint>
+    </xacro:if>
+  </xacro:unless>
 </robot>

File: xacro/ros2_control/interfaces.xacro (robot description, xacro)
@@ -6,37 +6,85 @@
 		<joint name="${prefix}joint1">
 			<command_interface name="position"/>
+			<command_interface name="velocity"/>
+			<command_interface name="effort"/>
+			<command_interface name="kp"/>
+			<command_interface name="kd"/>
 			<state_interface name="position"/>
 			<state_interface name="velocity"/>
 			<state_interface name="effort"/>
+			<param name="max_torque">21.0</param>
+			<param name="max_velocity">4.2</param>
+			<param name="kp">20.0</param>
+			<param name="kd">0.2</param>
 		</joint>
 		<joint name="${prefix}joint2">
 			<command_interface name="position"/>
+			<command_interface name="velocity"/>
+			<command_interface name="effort"/>
+			<command_interface name="kp"/>
+			<command_interface name="kd"/>
 			<state_interface name="position"/>
 			<state_interface name="velocity"/>
 			<state_interface name="effort"/>
+			<param name="max_torque">36.0</param>
+			<param name="max_velocity">5.0</param>
+			<param name="kp">30.0</param>
+			<param name="kd">0.3</param>
 		</joint>
 		<joint name="${prefix}joint3">
 			<command_interface name="position"/>
+			<command_interface name="velocity"/>
+			<command_interface name="effort"/>
+			<command_interface name="kp"/>
+			<command_interface name="kd"/>
 			<state_interface name="position"/>
 			<state_interface name="velocity"/>
 			<state_interface name="effort"/>
+			<param name="max_torque">36.0</param>
+			<param name="max_velocity">5.0</param>
+			<param name="kp">40.0</param>
+			<param name="kd">0.4</param>
 		</joint>
 		<joint name="${prefix}joint4">
 			<command_interface name="position"/>
+			<command_interface name="velocity"/>
+			<command_interface name="effort"/>
+			<command_interface name="kp"/>
+			<command_interface name="kd"/>
 			<state_interface name="position"/>
 			<state_interface name="velocity"/>
 			<state_interface name="effort"/>
+			<param name="max_torque">21.0</param>
+			<param name="max_velocity">4.2</param>
+			<param name="kp">20.0</param>
+			<param name="kd">0.2</param>
 		</joint>
 		<joint name="${prefix}joint5">
 			<command_interface name="position"/>
+			<command_interface name="velocity"/>
+			<command_interface name="effort"/>
+			<command_interface name="kp"/>
+			<command_interface name="kd"/>
 			<state_interface name="position"/>
 			<state_interface name="velocity"/>
 			<state_interface name="effort"/>
+			<param name="max_torque">10.0</param>
+			<param name="max_velocity">3.7</param>
+			<param name="kp">20.0</param>
+			<param name="kd">0.2</param>
 		</joint>
 		<joint name="${prefix}joint6">
 			<command_interface name="position"/>
+			<command_interface name="velocity"/>
+			<command_interface name="effort"/>
+			<command_interface name="kp"/>
+			<command_interface name="kd"/>
 			<state_interface name="position"/>
 			<state_interface name="velocity"/>
 			<state_interface name="effort"/>
+			<param name="max_torque">10.0</param>
+			<param name="max_velocity">3.7</param>
+			<param name="kp">20.0</param>
+			<param name="kd">0.2</param>
 		</joint>
 		<joint name="${prefix}gripper_joint">
@@ -47,12 +95,15 @@
 			<state_interface name="velocity"/>
 			<state_interface name="effort"/>
+			<param name="max_torque">0.5</param>
+			<param name="max_velocity">0.3</param>
+			<param name="kp">5.0</param>
+			<param name="kd">0.1</param>
 		</joint>
-		<xacro:if value="$(arg gazebo)">
-			<joint name="${prefix}gripper_joint2">
-				<state_interface name="position"/>
-				<state_interface name="velocity"/>
-				<state_interface name="effort"/>
-			</joint>
-		</xacro:if>
+		<!-- Mimic finger: state only (matches DualHardwareInterface 8-DoF-per-arm layout) -->
+		<joint name="${prefix}gripper_joint2">
+			<state_interface name="position"/>
+			<state_interface name="velocity"/>
+			<state_interface name="effort"/>
+		</joint>
 	</xacro:macro>
 </robot>

File: xacro/ros2_control/robot.xacro (robot description, xacro)
@@ -1,32 +1,110 @@
 <?xml version="1.0"?>
 <robot name="Panthera HT" xmlns:xacro="http://www.ros.org/wiki/xacro">
-  <link name="world"/>
-  <joint name="world_fixed" type="fixed">
-    <parent link="world"/>
-    <child link="base_link"/>
-  </joint>
+  <xacro:arg name="type" default="empty"/>
+  <xacro:arg name="control_mode" default="full_control"/>
+  <xacro:arg name="config_file"
+             default="$(find panthera_ros2_control)/external/motor_cpp/robot_param/Panthera.yaml"/>
+  <xacro:arg name="dual_config_file"
+             default="$(find panthera_ros2_control)/external/motor_cpp/robot_param/PantheraDual.yaml"/>
+  <xacro:property name="_type" value="$(arg type)"/>
+  <xacro:property name="_arm_config" value="single"/>
+  <xacro:if value="${_type == 'left'}">
+    <xacro:property name="_arm_config" value="left"/>
+  </xacro:if>
+  <xacro:if value="${_type == 'right'}">
+    <xacro:property name="_arm_config" value="right"/>
+  </xacro:if>
+  <xacro:if value="${_type == 'dual'}">
+    <xacro:property name="_arm_config" value="dual"/>
+  </xacro:if>
+  <!-- Select motor YAML: dual uses 14 motors; otherwise 7 -->
+  <xacro:property name="_config_file" value="$(arg config_file)"/>
+  <xacro:if value="${_arm_config == 'dual'}">
+    <xacro:property name="_config_file" value="$(arg dual_config_file)"/>
+  </xacro:if>
+  <xacro:if value="${_arm_config == 'single'}">
+    <link name="world"/>
+    <joint name="world_fixed" type="fixed">
+      <parent link="world"/>
+      <child link="base_link"/>
+    </joint>
+  </xacro:if>
   <xacro:include filename="$(find panthera_ht_description)/xacro/robot.xacro"/>
   <xacro:include filename="$(find panthera_ht_description)/xacro/ros2_control/interfaces.xacro"/>
-  <ros2_control name="panthera_ht_system" type="system">
-    <hardware>
-      <xacro:if value="${'$(arg ros2_control_hardware_type)' == 'gz'}">
-        <plugin>gz_ros2_control/GazeboSimSystem</plugin>
+  <!-- Real hardware: one PantheraHardwareInterface; motor count from config_file -->
+  <xacro:if value="${'$(arg ros2_control_hardware_type)' == 'real'}">
+    <ros2_control name="panthera_ht_system" type="system">
+      <hardware>
+        <plugin>panthera_ros2_control/PantheraHardwareInterface</plugin>
+        <param name="config_file">${_config_file}</param>
+        <param name="control_mode">$(arg control_mode)</param>
+        <param name="command_debug_enabled">false</param>
+        <param name="command_debug_period">1.0</param>
+        <param name="arm_velocity_filter_alpha">0.25</param>
+        <param name="arm_command_velocity_limit_scale">0.25</param>
+        <param name="arm_command_position_deadband">0.00001</param>
+        <param name="gripper_command_epsilon">0.0001</param>
+        <param name="gripper_rad_to_m">0.025</param>
+        <param name="shutdown_return_home">true</param>
+        <param name="shutdown_home">0.0, 0.0, 0.0, 0.0, 0.0, 0.0</param>
+        <param name="shutdown_home_timeout">3.5</param>
+        <param name="shutdown_home_tolerance">0.05</param>
+        <param name="shutdown_home_velocity">0.3</param>
+      </hardware>
+      <xacro:if value="${_arm_config == 'dual'}">
+        <xacro:panthera_ht_interfaces name="left"/>
+        <xacro:panthera_ht_interfaces name="right"/>
       </xacro:if>
-      <xacro:if value="${'$(arg ros2_control_hardware_type)' == 'mock_components'}">
-        <plugin>mock_components/GenericSystem</plugin>
+      <xacro:if value="${_arm_config == 'left'}">
+        <xacro:panthera_ht_interfaces name="left"/>
       </xacro:if>
-      <xacro:if value="${'$(arg ros2_control_hardware_type)' == 'isaac'}">
-        <plugin>topic_based_ros2_control/TopicBasedSystem</plugin>
-        <param name="joint_commands_topic">/isaac/joint_command</param>
-        <param name="joint_states_topic">/isaac/joint_states</param>
+      <xacro:if value="${_arm_config == 'right'}">
+        <xacro:panthera_ht_interfaces name="right"/>
       </xacro:if>
-    </hardware>
-    <xacro:panthera_ht_interfaces name=""/>
-  </ros2_control>
+      <xacro:if value="${_arm_config == 'single'}">
+        <xacro:panthera_ht_interfaces name=""/>
+      </xacro:if>
+    </ros2_control>
+  </xacro:if>
+  <xacro:unless value="${'$(arg ros2_control_hardware_type)' == 'real'}">
+    <ros2_control name="panthera_ht_system" type="system">
+      <hardware>
+        <xacro:if value="${'$(arg ros2_control_hardware_type)' == 'gz'}">
+          <plugin>gz_ros2_control/GazeboSimSystem</plugin>
+        </xacro:if>
+        <xacro:if value="${'$(arg ros2_control_hardware_type)' == 'mock_components'}">
+          <plugin>mock_components/GenericSystem</plugin>
+        </xacro:if>
+        <xacro:if value="${'$(arg ros2_control_hardware_type)' == 'isaac'}">
+          <plugin>topic_based_ros2_control/TopicBasedSystem</plugin>
+          <param name="joint_commands_topic">/isaac/joint_command</param>
+          <param name="joint_states_topic">/isaac/joint_states</param>
+        </xacro:if>
+      </hardware>
+      <xacro:if value="${_arm_config == 'dual'}">
+        <xacro:panthera_ht_interfaces name="left"/>
+        <xacro:panthera_ht_interfaces name="right"/>
+      </xacro:if>
+      <xacro:if value="${_arm_config == 'left'}">
+        <xacro:panthera_ht_interfaces name="left"/>
+      </xacro:if>
+      <xacro:if value="${_arm_config == 'right'}">
+        <xacro:panthera_ht_interfaces name="right"/>
+      </xacro:if>
+      <xacro:if value="${_arm_config == 'single'}">
+        <xacro:panthera_ht_interfaces name=""/>
+      </xacro:if>
+    </ros2_control>
+  </xacro:unless>
   <xacro:arg name="gazebo" default="false"/>
   <xacro:if value="$(arg gazebo)">
     <gazebo>
       <plugin filename="gz_ros2_control-system" name="gz_ros2_control::GazeboSimROS2ControlPlugin">
-        <parameters>$(find panthera_ht_description)/config/ros2_control/ros2_controllers.yaml</parameters>
+        <xacro:if value="${_arm_config == 'dual'}">
+          <parameters>$(find panthera_ht_description)/config/ros2_control/dual.yaml</parameters>
+        </xacro:if>
+        <xacro:unless value="${_arm_config == 'dual'}">
+          <parameters>$(find panthera_ht_description)/config/ros2_control/ros2_controllers.yaml</parameters>
+        </xacro:unless>
       </plugin>
     </gazebo>
