Commit message: fix: use package:// mesh paths in OCS2 URDF files.
Switch xacro mesh refs from file://$(find ...) to package://panthera_ht_description;
regenerate urdf/*.urdf and add scripts/generate_urdf.sh for export.

Co-authored-by: Cursor <cursoragent@cursor.com>

File: panthera_ht_description/urdf/panthera_ht.urdf (robot description, URDF)
Before this commit: robot Panthera HT, 10 links, 9 joints
Links:
- link base_link: geometry collision mesh filename=package://panthera_ht_description/meshes/base_link.glb; visual mesh filename=package://panthera_ht_description/meshes/base_link.glb
- link finger1: geometry collision mesh filename=package://panthera_ht_description/meshes/gripper_pad.glb; visual mesh filename=package://panthera_ht_description/meshes/gripper_pad.glb
- link finger2: geometry collision mesh filename=package://panthera_ht_description/meshes/gripper_pad.glb; visual mesh filename=package://panthera_ht_description/meshes/gripper_pad.glb
- link link1: geometry collision mesh filename=package://panthera_ht_description/meshes/link1.glb; visual mesh filename=package://panthera_ht_description/meshes/link1.glb
- link link2: geometry collision mesh filename=package://panthera_ht_description/meshes/link2.glb; visual mesh filename=package://panthera_ht_description/meshes/link2.glb
- link link3: geometry collision mesh filename=package://panthera_ht_description/meshes/link3.glb; visual mesh filename=package://panthera_ht_description/meshes/link3.glb
- link link4: geometry collision mesh filename=package://panthera_ht_description/meshes/link4.glb; visual mesh filename=package://panthera_ht_description/meshes/link4.glb
- link link5: geometry collision mesh filename=package://panthera_ht_description/meshes/link5.glb; visual mesh filename=package://panthera_ht_description/meshes/link5.glb
- link link6: geometry collision mesh filename=package://panthera_ht_description/meshes/link6.glb; visual mesh filename=package://panthera_ht_description/meshes/link6.glb

File: panthera_ht_description/urdf/panthera_ht_dual.urdf (robot description, URDF)
Before this commit: robot Panthera HT, 25 links, 24 joints
Links:
- link left_base_link: geometry collision mesh filename=package://panthera_ht_description/meshes/base_link.glb; visual mesh filename=package://panthera_ht_description/meshes/base_link.glb
- link left_finger1: geometry collision mesh filename=package://panthera_ht_description/meshes/gripper_pad.glb; visual mesh filename=package://panthera_ht_description/meshes/gripper_pad.glb
- link left_finger2: geometry collision mesh filename=package://panthera_ht_description/meshes/gripper_pad.glb; visual mesh filename=package://panthera_ht_description/meshes/gripper_pad.glb
- link left_link1: geometry collision mesh filename=package://panthera_ht_description/meshes/link1.glb; visual mesh filename=package://panthera_ht_description/meshes/link1.glb
- link left_link2: geometry collision mesh filename=package://panthera_ht_description/meshes/link2.glb; visual mesh filename=package://panthera_ht_description/meshes/link2.glb
- link left_link3: geometry collision mesh filename=package://panthera_ht_description/meshes/link3.glb; visual mesh filename=package://panthera_ht_description/meshes/link3.glb
- link left_link4: geometry collision mesh filename=package://panthera_ht_description/meshes/link4.glb; visual mesh filename=package://panthera_ht_description/meshes/link4.glb
- link left_link5: geometry collision mesh filename=package://panthera_ht_description/meshes/link5.glb; visual mesh filename=package://panthera_ht_description/meshes/link5.glb
- link left_link6: geometry collision mesh filename=package://panthera_ht_description/meshes/link6.glb; visual mesh filename=package://panthera_ht_description/meshes/link6.glb
- link right_base_link: geometry collision mesh filename=package://panthera_ht_description/meshes/base_link.glb; visual mesh filename=package://panthera_ht_description/meshes/base_link.glb
- link right_finger1: geometry collision mesh filename=package://panthera_ht_description/meshes/gripper_pad.glb; visual mesh filename=package://panthera_ht_description/meshes/gripper_pad.glb
- link right_finger2: geometry collision mesh filename=package://panthera_ht_description/meshes/gripper_pad.glb; visual mesh filename=package://panthera_ht_description/meshes/gripper_pad.glb
- link right_link1: geometry collision mesh filename=package://panthera_ht_description/meshes/link1.glb; visual mesh filename=package://panthera_ht_description/meshes/link1.glb
- link right_link2: geometry collision mesh filename=package://panthera_ht_description/meshes/link2.glb; visual mesh filename=package://panthera_ht_description/meshes/link2.glb
- link right_link3: geometry collision mesh filename=package://panthera_ht_description/meshes/link3.glb; visual mesh filename=package://panthera_ht_description/meshes/link3.glb
- link right_link4: geometry collision mesh filename=package://panthera_ht_description/meshes/link4.glb; visual mesh filename=package://panthera_ht_description/meshes/link4.glb
- link right_link5: geometry collision mesh filename=package://panthera_ht_description/meshes/link5.glb; visual mesh filename=package://panthera_ht_description/meshes/link5.glb
- link right_link6: geometry collision mesh filename=package://panthera_ht_description/meshes/link6.glb; visual mesh filename=package://panthera_ht_description/meshes/link6.glb

File: panthera_ht_description/urdf/panthera_ht_left.urdf (robot description, URDF)
Before this commit: robot Panthera HT, 15 links, 14 joints
Links:
- link left_base_link: geometry collision mesh filename=package://panthera_ht_description/meshes/base_link.glb; visual mesh filename=package://panthera_ht_description/meshes/base_link.glb
- link left_finger1: geometry collision mesh filename=package://panthera_ht_description/meshes/gripper_pad.glb; visual mesh filename=package://panthera_ht_description/meshes/gripper_pad.glb
- link left_finger2: geometry collision mesh filename=package://panthera_ht_description/meshes/gripper_pad.glb; visual mesh filename=package://panthera_ht_description/meshes/gripper_pad.glb
- link left_link1: geometry collision mesh filename=package://panthera_ht_description/meshes/link1.glb; visual mesh filename=package://panthera_ht_description/meshes/link1.glb
- link left_link2: geometry collision mesh filename=package://panthera_ht_description/meshes/link2.glb; visual mesh filename=package://panthera_ht_description/meshes/link2.glb
- link left_link3: geometry collision mesh filename=package://panthera_ht_description/meshes/link3.glb; visual mesh filename=package://panthera_ht_description/meshes/link3.glb
- link left_link4: geometry collision mesh filename=package://panthera_ht_description/meshes/link4.glb; visual mesh filename=package://panthera_ht_description/meshes/link4.glb
- link left_link5: geometry collision mesh filename=package://panthera_ht_description/meshes/link5.glb; visual mesh filename=package://panthera_ht_description/meshes/link5.glb
- link left_link6: geometry collision mesh filename=package://panthera_ht_description/meshes/link6.glb; visual mesh filename=package://panthera_ht_description/meshes/link6.glb

File: panthera_ht_description/urdf/panthera_ht_right.urdf (robot description, URDF)
Before this commit: robot Panthera HT, 15 links, 14 joints
Links:
- link right_base_link: geometry collision mesh filename=package://panthera_ht_description/meshes/base_link.glb; visual mesh filename=package://panthera_ht_description/meshes/base_link.glb
- link right_finger1: geometry collision mesh filename=package://panthera_ht_description/meshes/gripper_pad.glb; visual mesh filename=package://panthera_ht_description/meshes/gripper_pad.glb
- link right_finger2: geometry collision mesh filename=package://panthera_ht_description/meshes/gripper_pad.glb; visual mesh filename=package://panthera_ht_description/meshes/gripper_pad.glb
- link right_link1: geometry collision mesh filename=package://panthera_ht_description/meshes/link1.glb; visual mesh filename=package://panthera_ht_description/meshes/link1.glb
- link right_link2: geometry collision mesh filename=package://panthera_ht_description/meshes/link2.glb; visual mesh filename=package://panthera_ht_description/meshes/link2.glb
- link right_link3: geometry collision mesh filename=package://panthera_ht_description/meshes/link3.glb; visual mesh filename=package://panthera_ht_description/meshes/link3.glb
- link right_link4: geometry collision mesh filename=package://panthera_ht_description/meshes/link4.glb; visual mesh filename=package://panthera_ht_description/meshes/link4.glb
- link right_link5: geometry collision mesh filename=package://panthera_ht_description/meshes/link5.glb; visual mesh filename=package://panthera_ht_description/meshes/link5.glb
- link right_link6: geometry collision mesh filename=package://panthera_ht_description/meshes/link6.glb; visual mesh filename=package://panthera_ht_description/meshes/link6.glb

File: panthera_ht_description/xacro/gripper.xacro (robot description, xacro)
@@ -17,10 +17,10 @@
       <visual>
         <geometry>
-          <mesh filename="file://$(find panthera_ht_description)/meshes/gripper_pad.glb"/>
+          <mesh filename="package://panthera_ht_description/meshes/gripper_pad.glb"/>
         </geometry>
       </visual>
       <collision>
         <geometry>
-          <mesh filename="file://$(find panthera_ht_description)/meshes/gripper_pad.glb"/>
+          <mesh filename="package://panthera_ht_description/meshes/gripper_pad.glb"/>
         </geometry>
       </collision>
@@ -48,5 +48,5 @@
         <origin rpy="${PI} 0 0"/>
         <geometry>
-          <mesh filename="file://$(find panthera_ht_description)/meshes/gripper_pad.glb"/>
+          <mesh filename="package://panthera_ht_description/meshes/gripper_pad.glb"/>
         </geometry>
       </visual>
@@ -54,5 +54,5 @@
         <origin rpy="${PI} 0 0"/>
         <geometry>
-          <mesh filename="file://$(find panthera_ht_description)/meshes/gripper_pad.glb"/>
+          <mesh filename="package://panthera_ht_description/meshes/gripper_pad.glb"/>
         </geometry>
       </collision>

File: panthera_ht_description/xacro/panthera_ht.xacro (robot description, xacro)
@@ -5,5 +5,5 @@
     <xacro:property name="prefix" value="${name + '_' if name else ''}"/>
     <mujoco>
-      <compiler meshdir="../meshes/visual" balanceinertia="true" discardvisual="false"/>
+      <compiler meshdir="../meshes" balanceinertia="true" discardvisual="false"/>
     </mujoco>
     <!-- Base Link -->
@@ -22,10 +22,10 @@
       <visual>
         <geometry>
-          <mesh filename="file://$(find panthera_ht_description)/meshes/base_link.glb"/>
-        </geometry>
-      </visual>
-      <collision>
-        <geometry>
-          <mesh filename="file://$(find panthera_ht_description)/meshes/base_link.glb"/>
+          <mesh filename="package://panthera_ht_description/meshes/base_link.glb"/>
+        </geometry>
+      </visual>
+      <collision>
+        <geometry>
+          <mesh filename="package://panthera_ht_description/meshes/base_link.glb"/>
         </geometry>
       </collision>
@@ -46,10 +46,10 @@
       <visual>
         <geometry>
-          <mesh filename="file://$(find panthera_ht_description)/meshes/link1.glb"/>
-        </geometry>
-      </visual>
-      <collision>
-        <geometry>
-          <mesh filename="file://$(find panthera_ht_description)/meshes/link1.glb"/>
+          <mesh filename="package://panthera_ht_description/meshes/link1.glb"/>
+        </geometry>
+      </visual>
+      <collision>
+        <geometry>
+          <mesh filename="package://panthera_ht_description/meshes/link1.glb"/>
         </geometry>
       </collision>
@@ -77,10 +77,10 @@
       <visual>
         <geometry>
-          <mesh filename="file://$(find panthera_ht_description)/meshes/link2.glb"/>
-        </geometry>
-      </visual>
-      <collision>
-        <geometry>
-          <mesh filename="file://$(find panthera_ht_description)/meshes/link2.glb"/>
+          <mesh filename="package://panthera_ht_description/meshes/link2.glb"/>
+        </geometry>
+      </visual>
+      <collision>
+        <geometry>
+          <mesh filename="package://panthera_ht_description/meshes/link2.glb"/>
         </geometry>
       </collision>
@@ -108,10 +108,10 @@
       <visual>
         <geometry>
-          <mesh filename="file://$(find panthera_ht_description)/meshes/link3.glb"/>
-        </geometry>
-      </visual>
-      <collision>
-        <geometry>
-          <mesh filename="file://$(find panthera_ht_description)/meshes/link3.glb"/>
+          <mesh filename="package://panthera_ht_description/meshes/link3.glb"/>
+        </geometry>
+      </visual>
+      <collision>
+        <geometry>
+          <mesh filename="package://panthera_ht_description/meshes/link3.glb"/>
         </geometry>
       </collision>
@@ -139,10 +139,10 @@
       <visual>
         <geometry>
-          <mesh filename="file://$(find panthera_ht_description)/meshes/link4.glb"/>
-        </geometry>
-      </visual>
-      <collision>
-        <geometry>
-          <mesh filename="file://$(find panthera_ht_description)/meshes/link4.glb"/>
+          <mesh filename="package://panthera_ht_description/meshes/link4.glb"/>
+        </geometry>
+      </visual>
+      <collision>
+        <geometry>
+          <mesh filename="package://panthera_ht_description/meshes/link4.glb"/>
         </geometry>
       </collision>
@@ -170,10 +170,10 @@
       <visual>
         <geometry>
-          <mesh filename="file://$(find panthera_ht_description)/meshes/link5.glb"/>
-        </geometry>
-      </visual>
-      <collision>
-        <geometry>
-          <mesh filename="file://$(find panthera_ht_description)/meshes/link5.glb"/>
+          <mesh filename="package://panthera_ht_description/meshes/link5.glb"/>
+        </geometry>
+      </visual>
+      <collision>
+        <geometry>
+          <mesh filename="package://panthera_ht_description/meshes/link5.glb"/>
         </geometry>
       </collision>
@@ -201,10 +201,10 @@
       <visual>
         <geometry>
-          <mesh filename="file://$(find panthera_ht_description)/meshes/link6.glb"/>
-        </geometry>
-      </visual>
-      <collision>
-        <geometry>
-          <mesh filename="file://$(find panthera_ht_description)/meshes/link6.glb"/>
+          <mesh filename="package://panthera_ht_description/meshes/link6.glb"/>
+        </geometry>
+      </visual>
+      <collision>
+        <geometry>
+          <mesh filename="package://panthera_ht_description/meshes/link6.glb"/>
         </geometry>
       </collision>
