Commit message: fixed: "package://panthera_ht_description" to "file://$(find panthera_ht_description)" fixed: "$(find panthera_ros2_control)" to "$(find ht_ros2_control)" fixed: "controller_manager.update_rate" from "100" to "500"; "mpc_frequency" from "50" to "100" removed: urdfs

File: panthera_ht_description/xacro/gripper.xacro (robot description, xacro)
@@ -17,10 +17,10 @@
       <visual>
         <geometry>
-          <mesh filename="package://panthera_ht_description/meshes/gripper_pad.glb"/>
+          <mesh filename="file://$(find panthera_ht_description)/meshes/gripper_pad.glb"/>
         </geometry>
       </visual>
       <collision>
         <geometry>
-          <mesh filename="package://panthera_ht_description/meshes/gripper_pad.glb"/>
+          <mesh filename="file://$(find panthera_ht_description)/meshes/gripper_pad.glb"/>
         </geometry>
       </collision>
@@ -48,5 +48,5 @@
         <origin rpy="${PI} 0 0"/>
         <geometry>
-          <mesh filename="package://panthera_ht_description/meshes/gripper_pad.glb"/>
+          <mesh filename="file://$(find panthera_ht_description)/meshes/gripper_pad.glb"/>
         </geometry>
       </visual>
@@ -54,5 +54,5 @@
         <origin rpy="${PI} 0 0"/>
         <geometry>
-          <mesh filename="package://panthera_ht_description/meshes/gripper_pad.glb"/>
+          <mesh filename="file://$(find panthera_ht_description)/meshes/gripper_pad.glb"/>
         </geometry>
       </collision>

File: panthera_ht_description/xacro/panthera_ht.xacro (robot description, xacro)
@@ -22,10 +22,10 @@
       <visual>
         <geometry>
-          <mesh filename="package://panthera_ht_description/meshes/base_link.glb"/>
-        </geometry>
-      </visual>
-      <collision>
-        <geometry>
-          <mesh filename="package://panthera_ht_description/meshes/base_link.glb"/>
+          <mesh filename="file://$(find panthera_ht_description)/meshes/base_link.glb"/>
+        </geometry>
+      </visual>
+      <collision>
+        <geometry>
+          <mesh filename="file://$(find panthera_ht_description)/meshes/base_link.glb"/>
         </geometry>
       </collision>
@@ -46,10 +46,10 @@
       <visual>
         <geometry>
-          <mesh filename="package://panthera_ht_description/meshes/link1.glb"/>
-        </geometry>
-      </visual>
-      <collision>
-        <geometry>
-          <mesh filename="package://panthera_ht_description/meshes/link1.glb"/>
+          <mesh filename="file://$(find panthera_ht_description)/meshes/link1.glb"/>
+        </geometry>
+      </visual>
+      <collision>
+        <geometry>
+          <mesh filename="file://$(find panthera_ht_description)/meshes/link1.glb"/>
         </geometry>
       </collision>
@@ -77,10 +77,10 @@
       <visual>
         <geometry>
-          <mesh filename="package://panthera_ht_description/meshes/link2.glb"/>
-        </geometry>
-      </visual>
-      <collision>
-        <geometry>
-          <mesh filename="package://panthera_ht_description/meshes/link2.glb"/>
+          <mesh filename="file://$(find panthera_ht_description)/meshes/link2.glb"/>
+        </geometry>
+      </visual>
+      <collision>
+        <geometry>
+          <mesh filename="file://$(find panthera_ht_description)/meshes/link2.glb"/>
         </geometry>
       </collision>
@@ -108,10 +108,10 @@
       <visual>
         <geometry>
-          <mesh filename="package://panthera_ht_description/meshes/link3.glb"/>
-        </geometry>
-      </visual>
-      <collision>
-        <geometry>
-          <mesh filename="package://panthera_ht_description/meshes/link3.glb"/>
+          <mesh filename="file://$(find panthera_ht_description)/meshes/link3.glb"/>
+        </geometry>
+      </visual>
+      <collision>
+        <geometry>
+          <mesh filename="file://$(find panthera_ht_description)/meshes/link3.glb"/>
         </geometry>
       </collision>
@@ -139,10 +139,10 @@
       <visual>
         <geometry>
-          <mesh filename="package://panthera_ht_description/meshes/link4.glb"/>
-        </geometry>
-      </visual>
-      <collision>
-        <geometry>
-          <mesh filename="package://panthera_ht_description/meshes/link4.glb"/>
+          <mesh filename="file://$(find panthera_ht_description)/meshes/link4.glb"/>
+        </geometry>
+      </visual>
+      <collision>
+        <geometry>
+          <mesh filename="file://$(find panthera_ht_description)/meshes/link4.glb"/>
         </geometry>
       </collision>
@@ -170,10 +170,10 @@
       <visual>
         <geometry>
-          <mesh filename="package://panthera_ht_description/meshes/link5.glb"/>
-        </geometry>
-      </visual>
-      <collision>
-        <geometry>
-          <mesh filename="package://panthera_ht_description/meshes/link5.glb"/>
+          <mesh filename="file://$(find panthera_ht_description)/meshes/link5.glb"/>
+        </geometry>
+      </visual>
+      <collision>
+        <geometry>
+          <mesh filename="file://$(find panthera_ht_description)/meshes/link5.glb"/>
         </geometry>
       </collision>
@@ -201,10 +201,10 @@
       <visual>
         <geometry>
-          <mesh filename="package://panthera_ht_description/meshes/link6.glb"/>
-        </geometry>
-      </visual>
-      <collision>
-        <geometry>
-          <mesh filename="package://panthera_ht_description/meshes/link6.glb"/>
+          <mesh filename="file://$(find panthera_ht_description)/meshes/link6.glb"/>
+        </geometry>
+      </visual>
+      <collision>
+        <geometry>
+          <mesh filename="file://$(find panthera_ht_description)/meshes/link6.glb"/>
         </geometry>
       </collision>
