Commit message: 修复：重力补偿中质量错误偏大的问题； 调整了控制器参数

File: panthera_ht_description/xacro/panthera_ht.xacro (robot description, xacro)
@@ -189,13 +189,14 @@
     <link name="${prefix}link6">
       <inertial>
-        <origin xyz="0.06704625 0.00051731 1.674e-05"/>
-        <mass value="0.45"/>
-        <inertia
-            ixx="0.00107368"
-            ixy="-1.25e-05"
-            ixz="3e-07"
-            iyy="0.00068998"
-            iyz="2.517e-05"
-            izz="0.00167551"/>
+        <origin xyz="0.03658064204800879 -4.423599645544578e-05 -3.475443117333792e-05"/>
+        <mass value="0.1360375427712166"/>
+        <!-- 带手柄的质量为 0.1365xxx ,不带手柄为 0.1065xxx , 修改后清理缓存： rm -rf /tmp/ocs2_ros2/panthera_ht/  -->
+        <inertia
+            ixx="0.001164611195900086"
+            ixy="-1.2480891149780458e-05"
+            ixz="3.091643577865139e-07"
+            iyy="0.0007145219412767848"
+            iyz="2.5218349472216365e-05"
+            izz="0.001773387394908565"/>
       </inertial>
       <visual>

File: panthera_ht_description/xacro/ros2_control/interfaces.xacro (robot description, xacro)
@@ -97,6 +97,14 @@
 			<param name="max_torque">0.5</param>
 			<param name="max_velocity">0.3</param>
-			<param name="kp">5.0</param>
-			<param name="kd">0.1</param>
+			<!-- 拖动模式 (xacro_drag_mode:=true): 低刚度, 夹爪可掰动 -->
+			<xacro:if value="${'$(arg drag_mode)' == 'true'}">
+				<param name="kp">0.001</param>
+				<param name="kd">0.01</param>
+			</xacro:if>
+			<!-- 正常模式 (默认) -->
+			<xacro:unless value="${'$(arg drag_mode)' == 'true'}">
+				<param name="kp">5.0</param>
+				<param name="kd">0.1</param>
+			</xacro:unless>
 		</joint>
 	</xacro:macro>

File: panthera_ht_description/xacro/ros2_control/robot.xacro (robot description, xacro)
@@ -3,4 +3,6 @@
   <xacro:arg name="type" default="single"/>
   <xacro:arg name="control_mode" default="full_control"/>
+  <!-- 拖动模式: low-stiffness (xacro_drag_mode:=true) -->
+  <xacro:arg name="drag_mode" default="false"/>
   <xacro:arg name="config_file"
              default="$(find ht_ros2_control)/external/motor_cpp/robot_param/Panthera.yaml"/>
