Commit message: 新增：添加了左臂或右臂单独启动的 controller yaml ，现在可以单独启动实物左右臂

File: panthera_ht_description/xacro/robot.xacro (robot description, xacro)
@@ -25,48 +25,50 @@
     <xacro:property name="_arm_config" value="dual"/>
   </xacro:if>
+  <xacro:property name="_body_xyz" value="$(arg body_xyz)"/>
+  <xacro:property name="_body_rpy" value="$(arg body_rpy)"/>
+  <xacro:property name="_left_mount_xyz" value="$(arg left_mount_xyz)"/>
+  <xacro:property name="_left_mount_rpy" value="$(arg left_mount_rpy)"/>
+  <xacro:property name="_right_mount_xyz" value="$(arg right_mount_xyz)"/>
+  <xacro:property name="_right_mount_rpy" value="$(arg right_mount_rpy)"/>
+  <link name="world"/>
+  <joint name="base_joint" type="fixed">
+      <parent link="world"/>
+      <child link="base_link"/>
+    </joint>
   <!-- Single arm (legacy): root link is `base_link` -->
-  <xacro:if value="${_arm_config == 'single'}">
+  <xacro:if value="${_arm_config == 'single' or _arm_config == 'left' or _arm_config == 'right'}">
     <xacro:Arm name=""/>
   </xacro:if>
-  <!-- Left-only / Right-only / Dual arms: mount one or two prefixed arms on a shared body -->
-  <xacro:unless value="${_arm_config == 'single'}">
-    <link name="world"/>
+  <!-- Dual arms: mount one or two prefixed arms on a shared body -->
+  <xacro:if value="${_arm_config == 'dual'}">
     <link name="base_link"/>
     <link name="body_link"/>
     <link name="left_mount"/>
     <link name="right_mount"/>
-    <joint name="base_joint" type="fixed">
-      <parent link="world"/>
-      <child link="base_link"/>
-    </joint>
     <joint name="body_joint" type="fixed">
-      <origin xyz="$(arg body_xyz)" rpy="$(arg body_rpy)"/>
+      <origin xyz="${_body_xyz}" rpy="${_body_rpy}"/>
       <parent link="base_link"/>
       <child link="body_link"/>
     </joint>
     <joint name="left_mount_joint" type="fixed">
-      <origin xyz="$(arg left_mount_xyz)" rpy="$(arg left_mount_rpy)"/>
+      <origin xyz="${_left_mount_xyz}" rpy="${_left_mount_rpy}"/>
       <parent link="body_link"/>
       <child link="left_mount"/>
     </joint>
     <joint name="right_mount_joint" type="fixed">
-      <origin xyz="$(arg right_mount_xyz)" rpy="$(arg right_mount_rpy)"/>
+      <origin xyz="${_right_mount_xyz}" rpy="${_right_mount_rpy}"/>
       <parent link="body_link"/>
       <child link="right_mount"/>
     </joint>
-    <xacro:if value="${_arm_config == 'left' or _arm_config == 'dual'}">
-      <xacro:Arm name="left"/>
-      <joint name="left_arm_mount_joint" type="fixed">
-        <parent link="left_mount"/>
-        <child link="left_base_link"/>
-      </joint>
-    </xacro:if>
-    <xacro:if value="${_arm_config == 'right' or _arm_config == 'dual'}">
-      <xacro:Arm name="right"/>
-      <joint name="right_arm_mount_joint" type="fixed">
-        <parent link="right_mount"/>
-        <child link="right_base_link"/>
-      </joint>
-    </xacro:if>
-  </xacro:unless>
+    <xacro:Arm name="left"/>
+    <joint name="left_arm_mount_joint" type="fixed">
+      <parent link="left_mount"/>
+      <child link="left_base_link"/>
+    </joint>
+    <xacro:Arm name="right"/>
+    <joint name="right_arm_mount_joint" type="fixed">
+      <parent link="right_mount"/>
+      <child link="right_base_link"/>
+    </joint>
+  </xacro:if>
 </robot>

File: panthera_ht_description/xacro/ros2_control/robot.xacro (robot description, xacro)
@@ -5,10 +5,7 @@
   <!-- 控制模式: full_control、pd_control、position_velocity -->
   <xacro:arg name="control_mode" default="full_control"/>
-  <!-- 高擎 SDK 电机配置文件 -->
-  <xacro:arg name="config_file"
-             default="$(find ht_ros2_control)/external/motor_cpp/robot_param/Panthera.yaml"/>
-  <!-- 双高擎 SDK 电机双臂配置文件 -->
-  <xacro:arg name="dual_config_file"
-             default="$(find ht_ros2_control)/external/motor_cpp/robot_param/PantheraDual.yaml"/>
+  <!-- 高擎 SDK 电机配置文件；默认空 = 按 type 自动选择（见 _config_file 选择逻辑）
+       可通过 launch 参数 xacro_config_file:=<path> 显式覆盖 -->
+  <xacro:arg name="config_file" default=""/>
   <!-- 每臂 7 值 CSV（6 臂关节 + 夹爪）；dual 时拼接为 14 值 -->
   <xacro:arg name="max_torques" default="21.0, 36.0, 36.0, 21.0, 10.0, 10.0, 0.5"/>
@@ -23,8 +20,5 @@
        多套机械臂同机时，各启动指定自己的控制盒路径。 -->
   <xacro:arg name="usb_select" default="auto"/>
-  <xacro:property name="_max_torques" value="$(arg max_torques)"/>
-  <xacro:property name="_max_velocities" value="$(arg max_velocities)"/>
-  <xacro:property name="_joint_kp" value="$(arg joint_kp)"/>
-  <xacro:property name="_joint_kd" value="$(arg joint_kd)"/>
+  <!-- resolve arm composition from `type` (Tianji-style) -->
   <xacro:property name="_type" value="$(arg type)"/>
   <xacro:property name="_arm_config" value="single"/>
@@ -38,15 +32,38 @@
     <xacro:property name="_arm_config" value="dual"/>
   </xacro:if>
-  <!-- Select motor YAML: dual uses 14 motors; otherwise 7 -->
-  <xacro:property name="_config_file" value="$(arg config_file)"/>
+  <xacro:property name="_max_torques" value="$(arg max_torques)"/>
+  <xacro:property name="_max_velocities" value="$(arg max_velocities)"/>
+  <xacro:property name="_joint_kp" value="$(arg joint_kp)"/>
+  <xacro:property name="_joint_kd" value="$(arg joint_kd)"/>
+  <xacro:property name="_control_mode" value="$(arg control_mode)"/>
+  <xacro:property name="_config_file_override" value="$(arg config_file)"/>
+  <xacro:property name="_usb_select" value="$(arg usb_select)"/>
+  <xacro:property name="_gripper_kp" value="$(arg gripper_kp)"/>
+  <xacro:property name="_gripper_kd" value="$(arg gripper_kd)"/>
+  <xacro:property name="_ros2_control_hardware_type" value="$(arg ros2_control_hardware_type)"/>
+  <!-- Select motor YAML by type: single → Panthera.yaml, left → PantheraLeft.yaml,
+       right → PantheraRight.yaml (serial_id=2), dual → PantheraDual.yaml (14 motors).
+       显式设置 config_file（如 xacro_config_file:=）时优先使用。 -->
+  <!-- 默认配置文件 -->
+  <xacro:property name="_config_file"
+             value="$(find ht_ros2_control)/external/motor_cpp/robot_param/Panthera.yaml"/>
+  <!-- 左臂配置文件 -->
+  <xacro:if value="${_arm_config == 'left'}">
+    <xacro:property name="_config_file"
+               value="$(find ht_ros2_control)/external/motor_cpp/robot_param/PantheraLeft.yaml"/>
+  </xacro:if>
+  <!-- 右臂配置文件 -->
+  <xacro:if value="${_arm_config == 'right'}">
+    <xacro:property name="_config_file"
+               value="$(find ht_ros2_control)/external/motor_cpp/robot_param/PantheraRight.yaml"/>
+  </xacro:if>
+  <!-- 双臂配置文件 -->
   <xacro:if value="${_arm_config == 'dual'}">
-    <xacro:property name="_config_file" value="$(arg dual_config_file)"/>
+    <xacro:property name="_config_file"
+               value="$(find ht_ros2_control)/external/motor_cpp/robot_param/PantheraDual.yaml"/>
   </xacro:if>
-  <xacro:if value="${_arm_config == 'single'}">
-    <link name="world"/>
-    <joint name="world_fixed" type="fixed">
-      <parent link="world"/>
-      <child link="base_link"/>
-    </joint>
+  <!-- 显式覆盖配置文件 -->
+  <xacro:if value="${_config_file_override != ''}">
+    <xacro:property name="_config_file" value="${_config_file_override}"/>
   </xacro:if>
   <xacro:include filename="$(find panthera_ht_description)/xacro/robot.xacro"/>
@@ -54,11 +71,11 @@
   <!-- Real hardware: one PantheraHardwareInterface; motor count from config_file -->
   <!-- 真实的硬件：PantheraHardwareInterface -->
-  <xacro:if value="${'$(arg ros2_control_hardware_type)' == 'real'}">
+  <xacro:if value="${_ros2_control_hardware_type == 'real'}">
     <ros2_control name="panthera_ht_system" type="system">
       <hardware>
         <plugin>ht_ros2_control/PantheraHardwareInterface</plugin>
         <param name="config_file">${_config_file}</param>
-        <param name="usb_select">$(arg usb_select)</param>
-        <param name="control_mode">$(arg control_mode)</param>
+        <param name="usb_select">${_usb_select}</param>
+        <param name="control_mode">${_control_mode}</param>
         <param name="gripper_rad_to_m">0.025</param>
         <param name="shutdown_return_home">true</param>
@@ -71,6 +88,6 @@
         <param name="joint_kp">${_joint_kp + ', ' + _joint_kp if _arm_config == 'dual' else _joint_kp}</param>
         <param name="joint_kd">${_joint_kd + ', ' + _joint_kd if _arm_config == 'dual' else _joint_kd}</param>
-        <param name="gripper_kp">$(arg gripper_kp)</param>
-        <param name="gripper_kd">$(arg gripper_kd)</param>
+        <param name="gripper_kp">${_gripper_kp}</param>
+        <param name="gripper_kd">${_gripper_kd}</param>
       </hardware>
       <!-- command 、 state 接口 -->
@@ -79,11 +96,5 @@
         <xacro:panthera_ht_interfaces name="right"/>
       </xacro:if>
-      <xacro:if value="${_arm_config == 'left'}">
-        <xacro:panthera_ht_interfaces name="left"/>
-      </xacro:if>
-      <xacro:if value="${_arm_config == 'right'}">
-        <xacro:panthera_ht_interfaces name="right"/>
-      </xacro:if>
-      <xacro:if value="${_arm_config == 'single'}">
+      <xacro:if value="${_arm_config == 'single' or _arm_config == 'left' or _arm_config == 'right'}">
         <xacro:panthera_ht_interfaces name=""/>
       </xacro:if>
@@ -91,17 +102,17 @@
   </xacro:if>
   <!-- 非真实硬件：GazeboSimSystem、mock_components、TopicBasedSystem -->
-  <xacro:unless value="${'$(arg ros2_control_hardware_type)' == 'real'}">
+  <xacro:unless value="${_ros2_control_hardware_type == 'real'}">
     <ros2_control name="panthera_ht_system" type="system">
       <hardware>
         <!-- Gazebo -->
-        <xacro:if value="${'$(arg ros2_control_hardware_type)' == 'gz'}">
+        <xacro:if value="${_ros2_control_hardware_type == 'gz'}">
           <plugin>gz_ros2_control/GazeboSimSystem</plugin>
         </xacro:if>
         <!-- mock -->
-        <xacro:if value="${'$(arg ros2_control_hardware_type)' == 'mock_components'}">
+        <xacro:if value="${_ros2_control_hardware_type == 'mock_components'}">
           <plugin>mock_components/GenericSystem</plugin>
         </xacro:if>
         <!-- Isaac -->
-        <xacro:if value="${'$(arg ros2_control_hardware_type)' == 'isaac'}">
+        <xacro:if value="${_ros2_control_hardware_type == 'isaac'}">
           <plugin>topic_based_ros2_control/TopicBasedSystem</plugin>
           <param name="joint_commands_topic">/isaac/joint_command</param>
@@ -114,11 +125,5 @@
         <xacro:panthera_ht_interfaces name="right"/>
       </xacro:if>
-      <xacro:if value="${_arm_config == 'left'}">
-        <xacro:panthera_ht_interfaces name="left"/>
-      </xacro:if>
-      <xacro:if value="${_arm_config == 'right'}">
-        <xacro:panthera_ht_interfaces name="right"/>
-      </xacro:if>
-      <xacro:if value="${_arm_config == 'single'}">
+      <xacro:if value="${_arm_config == 'single' or _arm_config == 'left' or _arm_config == 'right'}">
         <xacro:panthera_ht_interfaces name=""/>
       </xacro:if>
@@ -126,5 +131,6 @@
   </xacro:unless>
   <xacro:arg name="gazebo" default="false"/>
-  <xacro:if value="$(arg gazebo)">
+  <xacro:property name="_gazebo" value="$(arg gazebo)"/>
+  <xacro:if value="${_gazebo == 'true'}">
     <gazebo>
       <plugin filename="gz_ros2_control-system" name="gz_ros2_control::GazeboSimROS2ControlPlugin">
