Commit message: 修改：将 hardware interface 关节接口数改为和电机数量一致， mimic 关节直接通过 urdf 中的 mimic 进行解析；

File: panthera_ht_description/xacro/ros2_control/interfaces.xacro (robot description, xacro)
@@ -100,10 +100,4 @@
 			<param name="kd">0.1</param>
 		</joint>
-		<!-- Mimic finger: state only (matches DualHardwareInterface 8-DoF-per-arm layout) -->
-		<joint name="${prefix}gripper_joint2">
-			<state_interface name="position"/>
-			<state_interface name="velocity"/>
-			<state_interface name="effort"/>
-		</joint>
 	</xacro:macro>
 </robot>

Commit message: 修改：删除了 command_interface 中的 kp kd；hardware 参数适配 ht-ros2-control/feature/remove_pkpd 的修改

File: panthera_ht_description/xacro/ros2_control/interfaces.xacro (robot description, xacro)
@@ -8,13 +8,7 @@
 			<command_interface name="velocity"/>
 			<command_interface name="effort"/>
-			<command_interface name="kp"/>
-			<command_interface name="kd"/>
 			<state_interface name="position"/>
 			<state_interface name="velocity"/>
 			<state_interface name="effort"/>
-			<param name="max_torque">21.0</param>
-			<param name="max_velocity">4.2</param>
-			<param name="kp">20.0</param>
-			<param name="kd">0.2</param>
 		</joint>
 		<joint name="${prefix}joint2">
@@ -22,13 +16,7 @@
 			<command_interface name="velocity"/>
 			<command_interface name="effort"/>
-			<command_interface name="kp"/>
-			<command_interface name="kd"/>
 			<state_interface name="position"/>
 			<state_interface name="velocity"/>
 			<state_interface name="effort"/>
-			<param name="max_torque">36.0</param>
-			<param name="max_velocity">5.0</param>
-			<param name="kp">30.0</param>
-			<param name="kd">0.3</param>
 		</joint>
 		<joint name="${prefix}joint3">
@@ -36,13 +24,7 @@
 			<command_interface name="velocity"/>
 			<command_interface name="effort"/>
-			<command_interface name="kp"/>
-			<command_interface name="kd"/>
 			<state_interface name="position"/>
 			<state_interface name="velocity"/>
 			<state_interface name="effort"/>
-			<param name="max_torque">36.0</param>
-			<param name="max_velocity">5.0</param>
-			<param name="kp">40.0</param>
-			<param name="kd">0.4</param>
 		</joint>
 		<joint name="${prefix}joint4">
@@ -50,13 +32,7 @@
 			<command_interface name="velocity"/>
 			<command_interface name="effort"/>
-			<command_interface name="kp"/>
-			<command_interface name="kd"/>
 			<state_interface name="position"/>
 			<state_interface name="velocity"/>
 			<state_interface name="effort"/>
-			<param name="max_torque">21.0</param>
-			<param name="max_velocity">4.2</param>
-			<param name="kp">20.0</param>
-			<param name="kd">0.2</param>
 		</joint>
 		<joint name="${prefix}joint5">
@@ -64,13 +40,7 @@
 			<command_interface name="velocity"/>
 			<command_interface name="effort"/>
-			<command_interface name="kp"/>
-			<command_interface name="kd"/>
 			<state_interface name="position"/>
 			<state_interface name="velocity"/>
 			<state_interface name="effort"/>
-			<param name="max_torque">10.0</param>
-			<param name="max_velocity">3.7</param>
-			<param name="kp">20.0</param>
-			<param name="kd">0.2</param>
 		</joint>
 		<joint name="${prefix}joint6">
@@ -78,13 +48,7 @@
 			<command_interface name="velocity"/>
 			<command_interface name="effort"/>
-			<command_interface name="kp"/>
-			<command_interface name="kd"/>
 			<state_interface name="position"/>
 			<state_interface name="velocity"/>
 			<state_interface name="effort"/>
-			<param name="max_torque">10.0</param>
-			<param name="max_velocity">3.7</param>
-			<param name="kp">20.0</param>
-			<param name="kd">0.2</param>
 		</joint>
 		<joint name="${prefix}gripper_joint">
@@ -95,16 +59,4 @@
 			<state_interface name="velocity"/>
 			<state_interface name="effort"/>
-			<param name="max_torque">0.5</param>
-			<param name="max_velocity">0.3</param>
-			<!-- 拖动模式 (xacro_drag_mode:=true): 低刚度, 夹爪可掰动 -->
-			<xacro:if value="${'$(arg drag_mode)' == 'true'}">
-				<param name="kp">0.001</param>
-				<param name="kd">0.01</param>
-			</xacro:if>
-			<!-- 正常模式 (默认) -->
-			<xacro:unless value="${'$(arg drag_mode)' == 'true'}">
-				<param name="kp">5.0</param>
-				<param name="kd">0.1</param>
-			</xacro:unless>
 		</joint>
 	</xacro:macro>

File: panthera_ht_description/xacro/ros2_control/robot.xacro (robot description, xacro)
@@ -1,12 +1,20 @@
 <?xml version="1.0"?>
 <robot name="Panthera HT" xmlns:xacro="http://www.ros.org/wiki/xacro">
+  <!-- 机器人类型: single、dual、left、right -->
   <xacro:arg name="type" default="single"/>
+  <!-- 控制模式: full_control、pd_control、position_velocity -->
   <xacro:arg name="control_mode" default="full_control"/>
-  <!-- 拖动模式: low-stiffness (xacro_drag_mode:=true) -->
-  <xacro:arg name="drag_mode" default="false"/>
+  <!-- 高擎 SDK 电机配置文件 -->
   <xacro:arg name="config_file"
              default="$(find ht_ros2_control)/external/motor_cpp/robot_param/Panthera.yaml"/>
+  <!-- 双高擎 SDK 电机双臂配置文件 -->
   <xacro:arg name="dual_config_file"
              default="$(find ht_ros2_control)/external/motor_cpp/robot_param/PantheraDual.yaml"/>
+  <!-- 每臂 7 值 CSV（6 臂关节 + 夹爪）；dual 时拼接为 14 值 -->
+  <xacro:property name="_max_torques" value="21.0, 36.0, 36.0, 21.0, 10.0, 10.0, 0.5"/>
+  <xacro:property name="_max_velocities" value="4.2, 5.0, 5.0, 4.2, 3.7, 3.7, 0.3"/>
+  <!-- 每臂 6 值 CSV（仅臂关节） -->
+  <xacro:property name="_joint_kp" value="20.0, 30.0, 40.0, 20.0, 20.0, 20.0"/>
+  <xacro:property name="_joint_kd" value="0.2, 0.3, 0.4, 0.2, 0.2, 0.2"/>
   <xacro:property name="_type" value="$(arg type)"/>
   <xacro:property name="_arm_config" value="single"/>
@@ -35,4 +43,5 @@
   <xacro:include filename="$(find panthera_ht_description)/xacro/ros2_control/interfaces.xacro"/>
   <!-- Real hardware: one PantheraHardwareInterface; motor count from config_file -->
+  <!-- 真实的硬件：PantheraHardwareInterface -->
   <xacro:if value="${'$(arg ros2_control_hardware_type)' == 'real'}">
     <ros2_control name="panthera_ht_system" type="system">
@@ -41,10 +50,4 @@
         <param name="config_file">${_config_file}</param>
         <param name="control_mode">$(arg control_mode)</param>
-        <param name="command_debug_enabled">false</param>
-        <param name="command_debug_period">1.0</param>
-        <param name="arm_velocity_filter_alpha">0.25</param>
-        <param name="arm_command_velocity_limit_scale">0.25</param>
-        <param name="arm_command_position_deadband">0.00001</param>
-        <param name="gripper_command_epsilon">0.0001</param>
         <param name="gripper_rad_to_m">0.025</param>
         <param name="shutdown_return_home">true</param>
@@ -53,5 +56,12 @@
         <param name="shutdown_home_tolerance">0.05</param>
         <param name="shutdown_home_velocity">0.3</param>
+        <param name="max_torques">${_max_torques + ', ' + _max_torques if _arm_config == 'dual' else _max_torques}</param>
+        <param name="max_velocities">${_max_velocities + ', ' + _max_velocities if _arm_config == 'dual' else _max_velocities}</param>
+        <param name="joint_kp">${_joint_kp + ', ' + _joint_kp if _arm_config == 'dual' else _joint_kp}</param>
+        <param name="joint_kd">${_joint_kd + ', ' + _joint_kd if _arm_config == 'dual' else _joint_kd}</param>
+        <param name="gripper_kp">5.0</param>
+        <param name="gripper_kd">0.1</param>
       </hardware>
+      <!-- command 、 state 接口 -->
       <xacro:if value="${_arm_config == 'dual'}">
         <xacro:panthera_ht_interfaces name="left"/>
@@ -69,13 +79,17 @@
     </ros2_control>
   </xacro:if>
+  <!-- 非真实硬件：GazeboSimSystem、mock_components、TopicBasedSystem -->
   <xacro:unless value="${'$(arg ros2_control_hardware_type)' == 'real'}">
     <ros2_control name="panthera_ht_system" type="system">
       <hardware>
+        <!-- Gazebo -->
         <xacro:if value="${'$(arg ros2_control_hardware_type)' == 'gz'}">
           <plugin>gz_ros2_control/GazeboSimSystem</plugin>
         </xacro:if>
+        <!-- mock -->
         <xacro:if value="${'$(arg ros2_control_hardware_type)' == 'mock_components'}">
           <plugin>mock_components/GenericSystem</plugin>
         </xacro:if>
+        <!-- Isaac -->
         <xacro:if value="${'$(arg ros2_control_hardware_type)' == 'isaac'}">
           <plugin>topic_based_ros2_control/TopicBasedSystem</plugin>
@@ -84,4 +98,5 @@
         </xacro:if>
       </hardware>
+      <!-- command 、 state 接口 -->
       <xacro:if value="${_arm_config == 'dual'}">
         <xacro:panthera_ht_interfaces name="left"/>
@@ -106,5 +121,5 @@
           <parameters>$(find panthera_ht_description)/config/ros2_control/dual.yaml</parameters>
         </xacro:if>
-        <xacro:unless value="${_arm_config == 'dual'}">
+        <xacro:unless value="${_arm_config == 'single'}">
           <parameters>$(find panthera_ht_description)/config/ros2_control/single.yaml</parameters>
         </xacro:unless>
