Commit message: 修复：调整了合适的参数

File: panthera_ht_description/xacro/ros2_control/robot.xacro (robot description, xacro)
@@ -15,6 +15,6 @@
   <xacro:property name="_max_velocities" value="4.2, 5.0, 5.0, 4.2, 3.7, 3.7, 0.3"/>
   <!-- 每臂 6 值 CSV（仅臂关节） -->
-  <xacro:property name="_joint_kp" value="20.0, 30.0, 40.0, 20.0, 20.0, 20.0"/>
-  <xacro:property name="_joint_kd" value="0.2, 0.3, 0.4, 0.2, 0.2, 0.2"/>
+  <xacro:property name="_joint_kp" value="40.0, 40.0, 40.0, 40.0, 40.0, 40.0"/>
+  <xacro:property name="_joint_kd" value="4.0, 4.0, 4.0, 4.0, 4.0, 4.0"/>
   <xacro:property name="_type" value="$(arg type)"/>
   <xacro:property name="_arm_config" value="single"/>
@@ -53,7 +53,7 @@
         <param name="shutdown_return_home">true</param>
         <param name="shutdown_home">0.0, 0.0, 0.0, 0.0, 0.0, 0.0</param>
-        <param name="shutdown_home_timeout">3.5</param>
-        <param name="shutdown_home_tolerance">0.05</param>
-        <param name="shutdown_home_velocity">0.3</param>
+        <param name="shutdown_home_timeout">3.0</param>
+        <param name="shutdown_home_tolerance">0.02</param>
+        <param name="shutdown_home_velocity">0.5</param>
         <param name="max_torques">${_max_torques + ', ' + _max_torques if _arm_config == 'dual' else _max_torques}</param>
         <param name="max_velocities">${_max_velocities + ', ' + _max_velocities if _arm_config == 'dual' else _max_velocities}</param>

Commit message: 修复：导出 hardware 参数为 arg

File: panthera_ht_description/xacro/ros2_control/robot.xacro (robot description, xacro)
@@ -12,9 +12,15 @@
              default="$(find ht_ros2_control)/external/motor_cpp/robot_param/PantheraDual.yaml"/>
   <!-- 每臂 7 值 CSV（6 臂关节 + 夹爪）；dual 时拼接为 14 值 -->
-  <xacro:property name="_max_torques" value="21.0, 36.0, 36.0, 21.0, 10.0, 10.0, 0.5"/>
-  <xacro:property name="_max_velocities" value="4.2, 5.0, 5.0, 4.2, 3.7, 3.7, 0.3"/>
-  <!-- 每臂 6 值 CSV（仅臂关节） -->
-  <xacro:property name="_joint_kp" value="40.0, 40.0, 40.0, 40.0, 40.0, 40.0"/>
-  <xacro:property name="_joint_kd" value="4.0, 4.0, 4.0, 4.0, 4.0, 4.0"/>
+  <xacro:arg name="max_torques" default="21.0, 36.0, 36.0, 21.0, 10.0, 10.0, 0.5"/>
+  <xacro:arg name="max_velocities" default="4.2, 5.0, 5.0, 4.2, 3.7, 3.7, 0.3"/>
+  <!-- 每臂 6 值 CSV（仅臂关节）；启动时可通过 launch 参数覆盖（xacro mappings） -->
+  <xacro:arg name="joint_kp" default="40.0, 40.0, 40.0, 40.0, 40.0, 40.0"/>
+  <xacro:arg name="joint_kd" default="4.0, 4.0, 4.0, 4.0, 4.0, 4.0"/>
+  <xacro:arg name="gripper_kp" default="5.0"/>
+  <xacro:arg name="gripper_kd" default="0.1"/>
+  <xacro:property name="_max_torques" value="$(arg max_torques)"/>
+  <xacro:property name="_max_velocities" value="$(arg max_velocities)"/>
+  <xacro:property name="_joint_kp" value="$(arg joint_kp)"/>
+  <xacro:property name="_joint_kd" value="$(arg joint_kd)"/>
   <xacro:property name="_type" value="$(arg type)"/>
   <xacro:property name="_arm_config" value="single"/>
@@ -60,6 +66,6 @@
         <param name="joint_kp">${_joint_kp + ', ' + _joint_kp if _arm_config == 'dual' else _joint_kp}</param>
         <param name="joint_kd">${_joint_kd + ', ' + _joint_kd if _arm_config == 'dual' else _joint_kd}</param>
-        <param name="gripper_kp">5.0</param>
-        <param name="gripper_kd">0.1</param>
+        <param name="gripper_kp">$(arg gripper_kp)</param>
+        <param name="gripper_kd">$(arg gripper_kd)</param>
       </hardware>
       <!-- command 、 state 接口 -->
